File: eagle/PSoC4Proto_Thermo/PSoC4Proto_Thermo.brd (EAGLE design)
At the start: 93.7 x 71.1 mm, 14 parts, among them IC2 PSOC4_PROTOTYPING_KIT, SW1 PUSH_SW_ALT

Commit message: Update: Eagle files
Parts:
- added JP3: GND_TP, pinhead:1X02
- added JP4: VBUS_TP, pinhead:1X02
- moved JP2 2.54 mm to (86.4, 57.1)
- moved SW1 2.54 mm to (86.4, 33.0)
- renumbered U$1 to IC1, U$2 to IC3
Connections:
- net +5V: now also SW1.2; no longer SW1.3
- net GND: now also JP3.1, JP3.2
- net VBUS: now also JP4.1, JP4.2
Routing:
- net GND: track 232.5 -> 243.7 mm
- net VBUS: track 27.9 -> 35.6 mm
- net V_TH: track 60.5 -> 64.1 mm
- net FOLLOWER_OUT: track 59.5 -> 62.0 mm
Changed lines of the file:
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@@
 <element name="IC2" library="mylib2" package="DIL44-8" value="PSOC4_PROTOTYPING_KIT" x="41.91" y="60.96" rot="R180"/>
 <element name="JP1" library="mylib2" package="MINI-USB_DIP" value="MINI-USB_DIP" x="81.28" y="12.7" rot="R270"/>
-<element name="JP2" library="pinhead" package="1X02" value="Thermistor" x="83.82" y="57.15" rot="R270"/>
+<element name="JP2" library="pinhead" package="1X02" value="Thermistor" x="86.36" y="57.15" rot="R270"/>
 <element name="R1" library="pot" package="B25P" value="10k" x="12.7" y="43.18" rot="R180"/>
 <element name="R2" library="rcl" package="0207/7" value="220" x="46.99" y="33.02" rot="R180"/>
 <element name="R3" library="rcl" package="0207/7" value="1k" x="59.69" y="43.18" rot="R180"/>
 <element name="R4" library="rcl" package="0207/7" value="10k" x="69.85" y="43.18"/>
-<element name="SW1" library="mylib2" package="PUSH_SW_ALT" value="PUSH_SW_ALT" x="86.36" y="30.48" rot="R90"/>
-<element name="U$1" library="mylib2" package="PSOC4-PROTO_USB-SERIAL_BRIDGE" value="PSOC4_USB-SERIAL_BRIDGE2" x="50.8" y="11.43" rot="R180"/>
-<element name="U$2" library="mylib2" package="TO226AA" value="TL431-INLINE" x="48.26" y="43.18" rot="R180"/>
+<element name="SW1" library="mylib2" package="PUSH_SW_ALT" value="PUSH_SW_ALT" x="86.36" y="33.02" rot="R90"/>
+<element name="IC1" library="mylib2" package="PSOC4-PROTO_USB-SERIAL_BRIDGE" value="PSOC4_USB-SERIAL_BRIDGE2" x="50.8" y="11.43" rot="R180"/>
+<element name="IC3" library="mylib2" package="TO226AA" value="TL431-INLINE" x="48.26" y="43.18" rot="R180"/>
 <element name="R5" library="rcl" package="0207/7" value="1k" x="69.85" y="2.54" rot="R180"/>
 <element name="LED1" library="led" package="LED3MM" value="Red" x="82.55" y="2.54" rot="R180"/>
+<element name="JP3" library="pinhead" package="1X02" value="GND_TP" x="85.09" y="48.26"/>
+<element name="JP4" library="pinhead" package="1X02" value="VBUS_TP" x="86.36" y="3.81" rot="R90"/>
 </elements>
 <signals>
 <signal name="DM">
 <contactref element="JP1" pad="4"/>
-<contactref element="U$1" pad="3"/>
+<contactref element="IC1" pad="3"/>
 <wire x1="81.28" y1="10.16" x2="78.74" y2="10.16" width="0.4064" layer="16"/>
 <wire x1="78.74" y1="10.16" x2="72.39" y2="10.16" width="0.4064" layer="1"/>
@@
 <signal name="DP">
 <contactref element="JP1" pad="3"/>
-<contactref element="U$1" pad="2"/>
+<contactref element="IC1" pad="2"/>
 <wire x1="81.28" y1="12.7" x2="78.74" y2="12.7" width="0.4064" layer="16"/>
 <wire x1="78.74" y1="12.7" x2="72.39" y2="12.7" width="0.4064" layer="1"/>
@@
 <signal name="GND">
 <contactref element="JP1" pad="1"/>
-<contactref element="U$1" pad="1"/>
+<contactref element="IC1" pad="1"/>
 <contactref element="IC2" pad="43"/>
 <contactref element="DIS1" pad="1"/>
 <contactref element="R1" pad="A"/>
 <contactref element="DIS1" pad="16"/>
-<contactref element="U$2" pad="2"/>
+<contactref element="IC3" pad="2"/>
 <contactref element="R4" pad="1"/>
 <contactref element="IC2" pad="5"/>
-<contactref element="U$1" pad="7"/>
+<contactref element="IC1" pad="7"/>
 <contactref element="C1" pad="-"/>
 <contactref element="R5" pad="2"/>
@@
 <wire x1="66.04" y1="15.24" x2="68.58" y2="17.78" width="0.4064" layer="16"/>
 <wire x1="68.58" y1="17.78" x2="78.74" y2="17.78" width="0.4064" layer="16"/>
+<contactref element="JP3" pad="1"/>
+<contactref element="JP3" pad="2"/>
+<wire x1="83.82" y1="48.26" x2="86.36" y2="48.26" width="0.4064" layer="16"/>
+<wire x1="76.2" y1="50.8" x2="81.28" y2="50.8" width="0.4064" layer="16"/>
+<wire x1="81.28" y1="50.8" x2="83.82" y2="48.26" width="0.4064" layer="16"/>
 </signal>
 <signal name="VBUS">
@@
 <wire x1="81.28" y1="7.62" x2="83.82" y2="7.62" width="0.4064" layer="16"/>
 <wire x1="83.82" y1="7.62" x2="83.82" y2="2.54" width="0.4064" layer="16"/>
-<wire x1="83.82" y1="27.94" x2="83.82" y2="7.62" width="0.4064" layer="16"/>
+<wire x1="83.82" y1="30.48" x2="83.82" y2="7.62" width="0.4064" layer="16"/>
+<contactref element="JP4" pad="2"/>
+<contactref element="JP4" pad="1"/>
+<wire x1="83.82" y1="2.54" x2="86.36" y2="2.54" width="0.4064" layer="16"/>
+<wire x1="86.36" y1="5.08" x2="86.36" y2="2.54" width="0.4064" layer="16"/>
 </signal>
 <signal name="+5V">
-<contactref element="SW1" pad="3"/>
+<contactref element="SW1" pad="2"/>
 <contactref element="IC2" pad="44"/>
 <contactref element="DIS1" pad="2"/>
@@
 <contactref element="R2" pad="1"/>
 <contactref element="R3" pad="1"/>
-<contactref element="U$1" pad="8"/>
+<contactref element="IC1" pad="8"/>
 <contactref element="C1" pad="+"/>
 <wire x1="10.16" y1="43.18" x2="9.91" y2="35.82" width="0.4064" layer="16"/>
@@
 <wire x1="68.58" y1="33.02" x2="68.58" y2="45.72" width="0.4064" layer="16"/>
 <wire x1="68.58" y1="45.72" x2="68.58" y2="48.26" width="0.4064" layer="16"/>
-<wire x1="83.82" y1="33.02" x2="68.58" y2="33.02" width="0.4064" layer="16"/>
 <wire x1="68.58" y1="48.26" x2="76.2" y2="48.26" width="0.4064" layer="16"/>
 <wire x1="63.5" y1="43.18" x2="63.5" y2="45.72" width="0.4064" layer="16"/>
@@
 <wire x1="50.8" y1="30.48" x2="48.51" y2="30.48" width="0.4064" layer="16"/>
 <wire x1="48.51" y1="30.48" x2="48.26" y2="30.73" width="0.4064" layer="16" curve="-90"/>
+<wire x1="83.82" y1="33.02" x2="68.58" y2="33.02" width="0.4064" layer="16"/>
 </signal>
 <signal name="RX">
 <contactref element="IC2" pad="24"/>
-<contactref element="U$1" pad="5"/>
+<contactref element="IC1" pad="5"/>
 <wire x1="17.78" y1="48.26" x2="17.78" y2="50.8" width="0.4064" layer="16"/>
 <wire x1="17.78" y1="50.8" x2="1.27" y2="50.8" width="0.4064" layer="16"/>
@@
 <signal name="TX">
 <contactref element="IC2" pad="23"/>
-<contactref element="U$1" pad="6"/>
+<contactref element="IC1" pad="6"/>
 <wire x1="15.24" y1="48.26" x2="5.08" y2="48.26" width="0.4064" layer="16"/>
 <wire x1="5.08" y1="48.26" x2="5.08" y2="12.7" width="0.4064" layer="16"/>
@@
 </signal>
 <signal name="FOLLOWER_IN">
-<contactref element="U$2" pad="3"/>
-<contactref element="U$2" pad="1"/>
+<contactref element="IC3" pad="3"/>
+<contactref element="IC3" pad="1"/>
 <contactref element="R3" pad="2"/>
 <contactref element="IC2" pad="35"/>
@@
 <contactref element="IC2" pad="42"/>
 <contactref element="IC2" pad="2"/>
-<wire x1="83.82" y1="55.88" x2="66.04" y2="55.88" width="0.4064" layer="16"/>
+<wire x1="86.36" y1="55.88" x2="66.04" y2="55.88" width="0.4064" layer="16"/>
 <wire x1="66.04" y1="55.88" x2="66.04" y2="68.58" width="0.4064" layer="16"/>
 <wire x1="50.8" y1="48.26" x2="50.8" y2="53.34" width="0.4064" layer="16"/>
@@
 <wire x1="60.96" y1="68.58" x2="63.5" y2="68.58" width="0.4064" layer="16"/>
 <wire x1="63.5" y1="68.58" x2="63.5" y2="66.04" width="0.4064" layer="16"/>
-<wire x1="63.5" y1="66.04" x2="83.82" y2="66.04" width="0.4064" layer="1"/>
-<wire x1="83.82" y1="58.42" x2="83.82" y2="66.04" width="0.4064" layer="16"/>
-<wire x1="86.36" y1="58.42" x2="83.82" y2="58.42" width="0.4064" layer="16"/>
+<wire x1="86.36" y1="58.42" x2="86.36" y2="60.96" width="0.4064" layer="16"/>
+<wire x1="88.9" y1="58.42" x2="86.36" y2="58.42" width="0.4064" layer="16"/>
 <via x="63.5" y="66.04" extent="1-16" drill="1" shape="square"/>
-<via x="83.82" y="66.04" extent="1-16" drill="1" shape="square"/>
-<wire x1="73.66" y1="43.18" x2="81.28" y2="43.18" width="0.4064" layer="16"/>
-<wire x1="86.36" y1="48.26" x2="86.36" y2="58.42" width="0.4064" layer="16"/>
-<wire x1="81.28" y1="43.18" x2="86.36" y2="48.26" width="0.4064" layer="16"/>
+<via x="86.36" y="60.96" extent="1-16" drill="1" shape="square"/>
+<wire x1="73.66" y1="43.18" x2="86.36" y2="43.18" width="0.4064" layer="16"/>
+<wire x1="88.9" y1="45.72" x2="88.9" y2="58.42" width="0.4064" layer="16"/>
+<wire x1="86.36" y1="43.18" x2="88.9" y2="45.72" width="0.4064" layer="16"/>
+<wire x1="63.5" y1="66.04" x2="81.28" y2="66.04" width="0.4064" layer="1"/>
+<wire x1="81.28" y1="66.04" x2="86.36" y2="60.96" width="0.4064" layer="1" curve="-90"/>
 </signal>
 <signal name="N$3">
